Commit message: Cleaned code and inserted gazebo extension in launch file

File: chefbot/chefbot_description/urdf/chefbot_base.urdf.xacro (robot description, xacro)
@@ -187,8 +187,6 @@
 	    </collision>
 	  </link>
-        <!-- Fixed because we never rotate it anyway, it is just for show -->
-        <!-- NOTE This may prevent gazebo from working with this model -->
-<!--
-	  <joint name="left_wheel_joint" type="fixed">
+        -->
+<!--	  <joint name="left_wheel_joint" type="fixed">
 	    <origin xyz="0 0.01905 0" rpy="0 0 0"/>
 	    <parent link="left_axle_link"/>
@@ -217,4 +215,5 @@
 	    </collision>
 	  </link>
+	-->
         <!-- Fixed because we never rotate it anyway, it is just for show -->
         <!-- NOTE This may prevent gazebo from working with this model -->
